File: circuit/hackerling.brd (EAGLE design)
At the start: 82.5 x 67.4 mm, 38 parts, among them IC1 MCP23017SP, IC2 MCP2300X/P, IC3 MIC5219BM5, U1 MMA8452Q, U2 LCD-16X2NOSILK, U3 ARDUINOR3-BPLACE

Commit message: fixing a few bugs, updating bom
Parts:
- renumbered C5 to C2, C6 to C3, U$1 to SW2, U$2 to IR1, U$5 to U5, U$7 to U7
Changed lines of the file:
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@@
 <layer number="48" name="Document" color="11" fill="1" visible="yes" active="yes"/>
 <layer number="49" name="Reference" color="7" fill="1" visible="no" active="yes"/>
-<layer number="50" name="dxf" color="7" fill="1" visible="no" active="yes"/>
-<layer number="51" name="tDocu" color="7" fill="1" visible="no" active="yes"/>
-<layer number="52" name="bDocu" color="7" fill="1" visible="no" active="yes"/>
+<layer number="50" name="dxf" color="7" fill="1" visible="yes" active="yes"/>
+<layer number="51" name="tDocu" color="7" fill="1" visible="yes" active="yes"/>
+<layer number="52" name="bDocu" color="7" fill="1" visible="yes" active="yes"/>
 <layer number="53" name="tGND_GNDA" color="7" fill="9" visible="no" active="no"/>
 <layer number="54" name="bGND_GNDA" color="1" fill="9" visible="no" active="no"/>
-<layer number="56" name="wert" color="7" fill="1" visible="no" active="yes"/>
+<layer number="56" name="wert" color="7" fill="1" visible="yes" active="yes"/>
 <layer number="91" name="Nets" color="2" fill="1" visible="no" active="no"/>
 <layer number="92" name="Busses" color="1" fill="1" visible="no" active="no"/>
@@
 </element>
 <element name="IC2" library="adafruit" package="DIL18" value="MCP2300X/P" x="53.48" y="39.32" rot="MR180"/>
-<element name="U$2" library="adafruit" package="PNA460XM" value="PNA460XM" x="68.61" y="65.26" rot="R180"/>
+<element name="IR1" library="adafruit" package="PNA460XM" value="PNA460XM" x="68.61" y="65.26" rot="R180"/>
 <element name="U$3" library="hackerscouts" package="ACCELEROMETER" value="ACCELEROMETER" x="24.47" y="46.62" smashed="yes" rot="MR0">
 <attribute name="NAME" x="31.8762" y="53.5488" size="1.27" layer="26" ratio="10" rot="MR0"/>
@@
 <element name="C1" library="resistor" package="C0603K" value="1uF" x="27.34" y="48.54" rot="R180"/>
 <element name="U1" library="hackerscouts" package="QFN-16(5X3)" value="MMA8452Q" x="20.41" y="50.4" rot="R90"/>
-<element name="C5" library="resistor" package="C0603K" value="0.1uF" x="24.17" y="47.63"/>
-<element name="C6" library="resistor" package="C0603K" value="4.7uF" x="23.87" y="51.36" rot="R90"/>
+<element name="C2" library="resistor" package="C0603K" value="0.1uF" x="24.17" y="47.63"/>
+<element name="C3" library="resistor" package="C0603K" value="4.7uF" x="23.87" y="51.36" rot="R90"/>
 <element name="R4" library="SparkFun" package="0603-RES" value="4k7" x="20.88" y="43.93"/>
-<element name="U$5" library="hackerscouts" package="VSSOP-8" value="PCA9306" x="26.24" y="44.82" rot="R270"/>
+<element name="U5" library="hackerscouts" package="VSSOP-8" value="PCA9306" x="26.24" y="44.82" rot="R270"/>
 <element name="R5" library="SparkFun" package="0603-RES" value="200K" x="29.68" y="45.73" rot="R270"/>
 <element name="U$6" library="hackerscouts" package="ACCELEROMETER" value="ACCELEROMETER" x="50.59" y="10.55" smashed="yes">
@@
 <attribute name="VALUE" x="42.97" y="2.295" size="1.27" layer="27"/>
 </element>
-<element name="U$7" library="hackerscouts" package="ALS_POT" value="POT" x="74.3646" y="9.5234" rot="R270"/>
+<element name="U7" library="hackerscouts" package="ALS_POT" value="POT" x="74.3646" y="9.5234" rot="R270"/>
 <element name="H4" library="holes" package="2,8" value="MOUNT-HOLE2.8" x="77.57" y="34.66"/>
 <element name="B1" library="hackerscouts" package="SWITCH_B3F-4000" value="" x="7.04" y="10.55" rot="R270"/>
@@
 <element name="B3" library="hackerscouts" package="SWITCH_B3F-4000" value="" x="33.11" y="10.44" rot="R90"/>
 <element name="B4" library="hackerscouts" package="SWITCH_B3F-4000" value="" x="20.01" y="10.5" rot="R90"/>
-<element name="U$1" library="hackerscouts" package="SWITCH_B13EH" value="SWITCH_B13EH" x="74.98" y="56.15" rot="R180"/>
+<element name="SW2" library="hackerscouts" package="SWITCH_B13EH" value="SWITCH_B13EH" x="74.98" y="56.15" rot="R180"/>
 <element name="U$8" library="hackerscouts" package="SML_POT" value="SML_POT" x="4.46" y="59.65" rot="MR270"/>
 </elements>
@@
 <contactref element="IC2" pad="9"/>
 <contactref element="IC1" pad="10"/>
-<contactref element="U$2" pad="2"/>
-<contactref element="U$2" pad="2"/>
+<contactref element="IR1" pad="2"/>
+<contactref element="IR1" pad="2"/>
 <contactref element="SERVO2" pad="3"/>
 <contactref element="SERVO1" pad="3"/>
 <contactref element="U$3" pad="4"/>
 <contactref element="IC3" pad="2"/>
-<contactref element="C5" pad="2"/>
+<contactref element="C2" pad="2"/>
 <contactref element="U1" pad="12"/>
 <contactref element="U1" pad="10"/>
@@
 <contactref element="IC3" pad="2"/>
 <contactref element="C1" pad="2"/>
-<contactref element="C6" pad="2"/>
-<contactref element="U$5" pad="P$1"/>
+<contactref element="C3" pad="2"/>
+<contactref element="U5" pad="P$1"/>
 <wire x1="19.06" y1="50.4" x2="19.91" y2="50.4" width="0.254" layer="1"/>
 <wire x1="19.91" y1="50.4" x2="19.91" y2="50.79" width="0.254" layer="1"/>
@@
 <wire x1="26.39" y1="47.1" x2="26.465" y2="47.485" width="0.4064" layer="1"/>
 <wire x1="26.465" y1="47.485" x2="26.465" y2="48.54" width="0.4064" layer="1"/>
-<contactref element="U$7" pad="P$1"/>
+<contactref element="U7" pad="P$1"/>
 <contactref element="U$6" pad="4"/>
 <wire x1="46.4" y1="13.06" x2="48.94" y2="13.06" width="0.4064" layer="16"/>
@@
 <vertex x="81.5" y="67.98"/>
 </polygon>
-<contactref element="U$1" pad="3"/>
+<contactref element="SW2" pad="3"/>
 <contactref element="U2" pad="1"/>
 <contactref element="U$8" pad="E"/>
@@
 <contactref element="IC2" pad="18"/>
 <contactref element="IC1" pad="9"/>
-<contactref element="U$2" pad="3"/>
-<contactref element="U$2" pad="3"/>
+<contactref element="IR1" pad="3"/>
+<contactref element="IR1" pad="3"/>
 <contactref element="U$3" pad="3"/>
 <contactref element="SW1" pad="6"/>
@@
 <wire x1="26.21" y1="45.82" x2="28.195" y2="46.815" width="0.3048" layer="1"/>
 <wire x1="28.195" y1="46.815" x2="28.215" y2="48.54" width="0.3048" layer="1"/>
-<contactref element="U$7" pad="P$3"/>
+<contactref element="U7" pad="P$3"/>
 <contactref element="U$6" pad="3"/>
 <via x="48.61" y="9.8" extent="1-16" drill="0.7"/>
@@
 <wire x1="23.83" y1="14.09" x2="20.1792" y2="14.09" width="0.6096" layer="16"/>
 <wire x1="20.1792" y1="14.09" x2="17.5208" y2="16.7484" width="0.6096" layer="16"/>
-<contactref element="U$1" pad="1"/>
+<contactref element="SW2" pad="1"/>
 <wire x1="74.98" y1="53.61" x2="69.7" y2="53.61" width="0.4064" layer="1"/>
 <wire x1="69.7" y1="53.61" x2="68.28" y2="52.19" width="0.4064" layer="1"/>
@@
 <contactref element="U3" pad="SCL"/>
 <contactref element="IC2" pad="1"/>
-<contactref element="U$5" pad="P$6"/>
+<contactref element="U5" pad="P$6"/>
 <contactref element="U$3" pad="2"/>
 <wire x1="27.43" y1="42.546" x2="27.43" y2="43.29" width="0.3048" layer="1"/>
@@
 <contactref element="U3" pad="SDA"/>
 <contactref element="IC2" pad="2"/>
-<contactref element="U$5" pad="P$5"/>
+<contactref element="U5" pad="P$5"/>
 <contactref element="U$3" pad="1"/>
 <wire x1="29.544" y1="43.48" x2="28.11" y2="43.48" width="0.3048" layer="1"/>
@@
 <signal name="POT">
 <contactref element="U3" pad="A3"/>
-<contactref element="U$7" pad="P$2"/>
+<contactref element="U7" pad="P$2"/>
 <wire x1="64.18" y1="13.06" x2="64.18" y2="12.17" width="0.4064" layer="1"/>
 <wire x1="64.18" y1="12.17" x2="68.202" y2="7.4114" width="0.4064" layer="1"/>
@@
 </signal>
 <signal name="IR_IN">
-<contactref element="U$2" pad="1"/>
+<contactref element="IR1" pad="1"/>
 <contactref element="U3" pad="D12"/>
 <wire x1="33.19" y1="67.23" x2="32.21" y2="66.19" width="0.254" layer="16"/>
@@
 <wire x1="71.42" y1="66.9" x2="72.29" y2="66.9" width="0.4064" layer="1"/>
 <wire x1="72.29" y1="66.9" x2="72.95" y2="66.24" width="0.4064" layer="1"/>
-<contactref element="U$1" pad="2"/>
+<contactref element="SW2" pad="2"/>
 <wire x1="72.95" y1="66.24" x2="72.95" y2="58.18" width="0.4064" layer="1"/>
 <wire x1="72.95" y1="58.18" x2="74.98" y2="56.15" width="0.4064" layer="1"/>
@@
 <signal name="3.3V">
 <contactref element="IC3" pad="5"/>
-<contactref element="U$5" pad="P$2"/>
-<contactref element="C6" pad="1"/>
+<contactref element="U5" pad="P$2"/>
+<contactref element="C3" pad="1"/>
 <contactref element="U1" pad="14"/>
 <contactref element="U1" pad="1"/>
@@
 </signal>
 <signal name="5V">
-<contactref element="U$5" pad="P$7"/>
+<contactref element="U5" pad="P$7"/>
 <contactref element="R5" pad="2"/>
 <wire x1="29.68" y1="44.88" x2="29.95" y2="44.72" width="0.254" layer="1"/>
@@
 </signal>
 <signal name="SCL_3">
-<contactref element="U$5" pad="P$3"/>
+<contactref element="U5" pad="P$3"/>
 <contactref element="U1" pad="4"/>
 <contactref element="R3" pad="1"/>
@@
 </signal>
 <signal name="SDA_3">
-<contactref element="U$5" pad="P$4"/>
+<contactref element="U5" pad="P$4"/>
 <contactref element="U1" pad="6"/>
 <contactref element="R4" pad="1"/>
@@
 <signal name="N$25">
 <contactref element="U1" pad="2"/>
-<contactref element="C5" pad="1"/>
+<contactref element="C2" pad="1"/>
 <wire x1="20.91" y1="49.05" x2="20.91" y2="47.69" width="0.254" layer="1"/>
 <wire x1="20.91" y1="47.69" x2="23.295" y2="47.63" width="0.254" layer="1"/>
 </signal>
 <signal name="N$27">
-<contactref element="U$5" pad="P$8"/>
+<contactref element="U5" pad="P$8"/>
 <contactref element="R5" pad="1"/>
 <wire x1="27.69" y1="45.57" x2="28.19" y2="45.57" width="0.254" layer="1"/>
