File: circuit/hackerling.sch (EAGLE design)
At the start: 16 parts, among them IC1 MCP23017SP, IC2 MCP2300X/P, U2 LCD-16X2NOSILK, U3 ARDUINOR3-BPLACE

Commit message: arranging the hackerling circuit, added accelerometer layout
Parts:
- added C1: 1uF, resistor:C-USC0603K
- added C5: 0.1uF, resistor:C-USC0603K
- added C6: 4.7uF, resistor:C-USC0603K
- added H1, H2, H3: MOUNT-HOLE3.2, holes:MOUNT-HOLE3.2
- added IC3: MIC5219BM5, v-reg-micrel:MIC5219BM5
- added R3, R4: 4k7, SparkFun:RESISTOR0603-RES
- added R5: 200K, SparkFun:RESISTOR0603-RES
- added S1, S3, S4: (no value), switch-omron:40-XX
- added S6: SWITCH-DPDTOS, SparkFun:SWITCH-DPDTOS
- added SERVO1, SERVO2: (no value), SparkFun:M03LOCK
- added U$3, U$6: ACCELEROMETER, hackerscouts:ACCELEROMETER
- added U$5: PCA9306, hackerscouts:PCA9306
- added U1: MMA8452Q, hackerscouts:MMA8452Q
- S2: value SWITCH-DPDTOS -> (none); device SparkFun:SWITCH-DPDTOS -> switch-omron:40-XX; MF (none) -> OMRON COMPONENTS USA; MPN (none) -> B3F-4000; OC_FARNELL (none) -> 176434; OC_NEWARK (none) -> 36K3105
Connections:
- removed net IR_OUT: LED1.C, LED2.C, U3.D5
- removed net N$11 (its old number): IC1.GPA5, U2.RS
- removed net N$24 (its old number): DZ1-7.A, RN3.8
- removed net N$28: SW1.3, U3.D1
- removed net N$29: SW1.4, U3.D0
- new net 3.3V: C6.1, IC3.OUT, R3.2, R4.2, U$5.VCC1, U1.VDD, U1.VDDIO
- new net 5V: R5.2, U$5.VCC2
- new net A_INT1: U$3.INT1, U1.INT1, U3.D3
- new net A_INT2: U$3.INT2, U1.INT2, U3.D2
- new net BTN1: S1.P, U3.D4
- new net BTN2: S2.P1, U3.D7
- new net BTN3: S3.P, U3.D0
- new net BTN4: S4.P1, U3.D1
- new net DIP1: IC2.GP5, SW1.2
- new net DIP2: IC2.GP6, SW1.3
- new net DIP3: IC2.GP7, SW1.4
- new net IR_OUT1: LED1.C, U3.D5
- new net IR_OUT2: LED2.C, U3.D6
- new net N$10: IC1.GPA7, U2.RS
- new net N$17: DZ1-10.A, RN4.5
- new net SCL1: U$3.SCL, U3.SCL@1
- new net SCL_3: R3.1, U$5.SCL1, U1.SCL
- new net SDA1: U$3.SDA, U3.SDA@1
- new net SDA_3: R4.1, U$5.SDA1, U1.SDA
- new net SVO1: SERVO1.1, U3.D9
- new net SVO2: SERVO2.1, U3.D10
- new net SWITCH: S6.2, U3.D13
- net GND: now also C1.2, C5.2, C6.2, IC3.GND, SERVO1.3, SERVO2.3, U$3.GND, U$5.GND, U1.GND, U1.GND@1, U1.GND@2, U1.SAO
- net IR_IN: now also U3.D12; no longer U3.D7
- net N$12: now also DZ1-7.A; no longer DZ1-8.A
- net N$13: now also DZ1-8.A; no longer DZ1-9.A
- net N$14: now also DZ1-9.A; no longer DZ1-10.A
- net N$16: now also RN3.8; no longer RN4.5
- net N$18: now also RN3.7; no longer RN3.2
- net N$19: now also RN3.6; no longer RN3.3
- net N$20: now also RN3.5; no longer RN3.4
- net N$21: now also RN3.4; no longer RN3.5
- net N$22: now also RN3.3; no longer RN3.6
- net N$23: now also RN3.2; no longer RN3.7
- net N$25: now also C5.1, U1.BYP; no longer U3.D12
- net N$26: now also U3.D8; no longer U3.D3
- net N$27: now also R5.1, U$5.EN; no longer SW1.2, U3.D2
- net N$9: now also IC1.GPA5; no longer IC1.GPA7
- net SCL: now also U$5.SCL2
- net SDA: now also U$5.SDA2
- net VCC: now also C1.1, IC3.EN, IC3.IN, S1.S, S2.S1, S3.S1, S4.S1, S6.1, SERVO1.2, SERVO2.2, SW1.5, SW1.6, SW1.7, SW1.8, U$3.+5V
Other:
- note added: "Check servo pinout"
- moved on the sheet: LED1, RN3, SG1, SW1

Commit message: still arranging, about to rotate and shift parts
Connections:
- net SCL: now also U$3.SCL
- net SCL1: no longer U$3.SCL
- net SDA: now also U$3.SDA
- net SDA1: no longer U$3.SDA
Other:
- moved on the sheet: U$6
Changed lines of the file:
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@@
 <instance part="R5" gate="G$1" x="370.84" y="91.44" rot="R90"/>
 <instance part="P+15" gate="G$1" x="426.72" y="58.42"/>
-<instance part="U$6" gate="G$1" x="-43.18" y="-25.4" rot="MR0"/>
+<instance part="U$6" gate="G$1" x="-40.64" y="-12.7" rot="MR0"/>
 </instances>
 <busses>
@@
 <pinref part="U$5" gate="G$1" pin="SCL2"/>
 </segment>
+<segment>
+<pinref part="U$3" gate="G$1" pin="SCL"/>
+<wire x1="-30.48" y1="33.02" x2="-41.91" y2="33.02" width="0.1524" layer="91"/>
+<label x="-39.37" y="33.02" size="1.778" layer="95"/>
+</segment>
 </net>
 <net name="SDA" class="0">
@@
 <label x="416.56" y="76.2" size="1.778" layer="95"/>
 <pinref part="U$5" gate="G$1" pin="SDA2"/>
+</segment>
+<segment>
+<pinref part="U$3" gate="G$1" pin="SDA"/>
+<wire x1="-30.48" y1="30.48" x2="-41.91" y2="30.48" width="0.1524" layer="91"/>
+<label x="-39.37" y="30.48" size="1.778" layer="95"/>
 </segment>
 </net>
@@
 <net name="SCL1" class="0">
 <segment>
-<pinref part="U$3" gate="G$1" pin="SCL"/>
-<wire x1="-30.48" y1="33.02" x2="-41.91" y2="33.02" width="0.1524" layer="91"/>
-<label x="-39.37" y="33.02" size="1.778" layer="95"/>
-</segment>
-<segment>
 <pinref part="U3" gate="G$1" pin="SCL@1"/>
 <wire x1="85.09" y1="58.42" x2="100.33" y2="58.42" width="0.1524" layer="91"/>
@@
 <net name="SDA1" class="0">
 <segment>
-<pinref part="U$3" gate="G$1" pin="SDA"/>
-<wire x1="-30.48" y1="30.48" x2="-41.91" y2="30.48" width="0.1524" layer="91"/>
-<label x="-39.37" y="30.48" size="1.778" layer="95"/>
-</segment>
-<segment>
 <pinref part="U3" gate="G$1" pin="SDA@1"/>

Commit message: circuit state as of barebones order BOM is out of date still.... Just copied hackerling_a back to hackerling.
Parts:
- removed S1, S2, S3, S4: (no value), switch-omron:40-XX
- removed S6: SWITCH-DPDTOS, SparkFun:SWITCH-DPDTOS
- added B1, B2, B3, B4: (no value), hackerscouts:SWITCH_BCF-4000
- added H4: MOUNT-HOLE2.8, holes:MOUNT-HOLE2.8
- added U$7: POT, hackerscouts:POT
- added U$8: SML_POT, hackerscouts:SML_POT
- U$1: value (none) -> SWITCH_B13EH; device SparkFun:POT -> hackerscouts:SWITCH_B13EH
Connections:
- removed net N$14: DZ1-9.A, RN4.4
- removed net N$19: DZ1-2.A, RN3.6
- removed net N$24: LED2.A, RN4.6
- removed net N$26: SW1.1, U3.D8
- new net BACKLIGHT: SW1.4, U2.K, U3.D8
- new net N$28: DZ1-7.A, RN4.7
- new net N$29: DZ1-8.A, RN4.6
- new net N$30: DZ1-9.A, RN4.5
- new net N$31: DZ1-10.A, RN4.4
- net A_INT1: now also U$6.INT1
- net A_INT2: now also U$6.INT2
- net BARGRAPH0: now also IC2.GP0; no longer IC1.GPA0
- net BARGRAPH1: now also IC2.GP1; no longer IC1.GPA1
- net BARGRAPH2: now also IC2.GP2; no longer IC1.GPA2
- net BARGRAPH3: now also IC2.GP3; no longer IC1.GPA3
- net BARGRAPH4: now also IC2.GP4; no longer IC1.GPA4
- net BARGRAPH5: now also IC1.GPA0; no longer IC2.GP0
- net BARGRAPH6: now also IC1.GPA1; no longer IC2.GP1
- net BARGRAPH7: now also IC1.GPA2; no longer IC2.GP2
- net BARGRAPH8: now also IC1.GPA3; no longer IC2.GP3
- net BARGRAPH9: now also IC1.GPA4; no longer IC2.GP4
- net BTN1: now also B1.P; no longer S1.P
- net BTN2: now also B2.P; no longer S2.P1
- net BTN3: now also B3.P; no longer S3.P
- net BTN4: now also B4.P1; no longer S4.P1
- net DIP1: now also SW1.1; no longer SW1.2
- net DIP2: now also SW1.2; no longer SW1.3
- net DIP3: now also SW1.3; no longer SW1.4
- net GND: now also SW1.5, U$1.3, U$6.GND, U$7.A, U$8.E, U2.VSS; no longer U$1.A, U2.VDD
- net N$12: now also LED2.A, RN3.2; no longer DZ1-7.A, RN4.2
- net N$13: now also U$8.S, U2.VO; no longer DZ1-8.A, RN4.3
- net N$16: now also RN3.3; no longer RN3.8
- net N$17: now also DZ1-2.A, RN3.5; no longer DZ1-10.A, RN4.5
- net N$18: now also RN3.4; no longer RN3.7
- net N$20: now also RN3.6; no longer RN3.5
- net N$21: now also RN3.7; no longer RN3.4
- net N$22: now also RN3.8; no longer RN3.3
- net N$23: now also RN4.8; no longer RN3.2
- net POT: now also U$7.S; no longer U$1.S
- net SCL1: now also U$6.SCL
- net SDA1: now also U$6.SDA
- net SWITCH: now also U$1.2; no longer S6.2
- net VCC: now also B1.S, B2.S1, B3.S1, B4.S1, U$1.1, U$6.+5V, U$7.E, U$8.A, U2.A, U2.VDD; no longer S1.S, S2.S1, S3.S1, S4.S1, S6.1, SW1.5, U$1.E
Other:
- moved on the sheet: LED2, RN4

Commit message: fixing a few bugs, updating bom
Parts:
- removed U$1: SWITCH_B13EH, hackerscouts:SWITCH_B13EH
- added SW2: SWITCH_B13EH, hackerscouts:SWITCH_B13EH
- renumbered C5 to C2, C6 to C3, U$2 to IR1, U$5 to U5, U$7 to U7
Connections:
- net GND: now also SW2.3; no longer U$1.3
- net SWITCH: now also SW2.2; no longer U$1.2
- net VCC: now also SW2.1; no longer U$1.1
Changed lines of the file:
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@@
 <part name="P+6" library="supply1" deviceset="VCC" device=""/>
 <part name="P+7" library="supply1" deviceset="VCC" device=""/>
-<part name="U$2" library="adafruit" deviceset="PNA460XM" device=""/>
+<part name="IR1" library="adafruit" deviceset="PNA460XM" device=""/>
 <part name="GND9" library="supply1" deviceset="GND" device=""/>
 <part name="P+8" library="supply1" deviceset="VCC" device=""/>
@@
 <part name="P+14" library="SparkFun" deviceset="3.3V" device=""/>
 <part name="U$4" library="SparkFun" deviceset="5V" device=""/>
-<part name="C5" library="resistor" deviceset="C-US" device="C0603K" value="0.1uF"/>
-<part name="C6" library="resistor" deviceset="C-US" device="C0603K" value="4.7uF"/>
+<part name="C2" library="resistor" deviceset="C-US" device="C0603K" value="0.1uF"/>
+<part name="C3" library="resistor" deviceset="C-US" device="C0603K" value="4.7uF"/>
 <part name="R4" library="SparkFun" deviceset="RESISTOR" device="0603-RES" value="4k7"/>
-<part name="U$5" library="hackerscouts" deviceset="PCA9306" device=""/>
+<part name="U5" library="hackerscouts" deviceset="PCA9306" device=""/>
 <part name="R5" library="SparkFun" deviceset="RESISTOR" device="0603-RES" value="200K"/>
 <part name="P+15" library="SparkFun" deviceset="3.3V" device=""/>
 <part name="U$6" library="hackerscouts" deviceset="ACCELEROMETER" device=""/>
-<part name="U$7" library="hackerscouts" deviceset="POT" device=""/>
+<part name="U7" library="hackerscouts" deviceset="POT" device=""/>
 <part name="P+16" library="supply1" deviceset="VCC" device=""/>
 <part name="GND17" library="supply1" deviceset="GND" device=""/>
@@
 <part name="B3" library="hackerscouts" deviceset="SWITCH_BCF-4000" device=""/>
 <part name="B4" library="hackerscouts" deviceset="SWITCH_BCF-4000" device=""/>
-<part name="U$1" library="hackerscouts" deviceset="SWITCH_B13EH" device=""/>
+<part name="SW2" library="hackerscouts" deviceset="SWITCH_B13EH" device=""/>
 <part name="GND18" library="supply1" deviceset="GND" device=""/>
 <part name="U$8" library="hackerscouts" deviceset="SML_POT" device=""/>
@@
 <instance part="P+6" gate="VCC" x="129.54" y="71.12"/>
 <instance part="P+7" gate="VCC" x="190.5" y="86.36"/>
-<instance part="U$2" gate="G$1" x="-38.1" y="109.22"/>
+<instance part="IR1" gate="G$1" x="-38.1" y="109.22"/>
 <instance part="GND9" gate="1" x="-20.32" y="99.06"/>
 <instance part="P+8" gate="VCC" x="-10.16" y="106.68"/>
@@
 <instance part="P+14" gate="G$1" x="386.08" y="99.06"/>
 <instance part="U$4" gate="G$1" x="398.78" y="101.6"/>
-<instance part="C5" gate="G$1" x="381" y="35.56"/>
-<instance part="C6" gate="G$1" x="429.26" y="50.8"/>
+<instance part="C2" gate="G$1" x="381" y="35.56"/>
+<instance part="C3" gate="G$1" x="429.26" y="50.8"/>
 <instance part="R4" gate="G$1" x="447.04" y="43.18" rot="R90"/>
-<instance part="U$5" gate="G$1" x="396.24" y="83.82"/>
+<instance part="U5" gate="G$1" x="396.24" y="83.82"/>
 <instance part="R5" gate="G$1" x="370.84" y="91.44" rot="R90"/>
 <instance part="P+15" gate="G$1" x="426.72" y="58.42"/>
 <instance part="U$6" gate="G$1" x="-40.64" y="-12.7" rot="MR0"/>
-<instance part="U$7" gate="G$1" x="50.8" y="86.36"/>
+<instance part="U7" gate="G$1" x="50.8" y="86.36"/>
 <instance part="P+16" gate="VCC" x="-22.86" y="2.54"/>
 <instance part="GND17" gate="1" x="-50.8" y="-17.78" rot="MR0"/>
@@
 <instance part="B3" gate="G$1" x="-91.44" y="15.24"/>
 <instance part="B4" gate="G$1" x="-78.74" y="15.24"/>
-<instance part="U$1" gate="G$1" x="-50.8" y="45.72"/>
+<instance part="SW2" gate="G$1" x="-63.5" y="45.72"/>
 <instance part="GND18" gate="1" x="-40.64" y="40.64" rot="MR0"/>
 <instance part="U$8" gate="G$1" x="180.34" y="68.58" rot="MR180"/>
@@
 <pinref part="GND6" gate="1" pin="GND"/>
 <wire x1="60.96" y1="76.2" x2="60.96" y2="78.74" width="0.1524" layer="91"/>
-<pinref part="U$7" gate="G$1" pin="A"/>
+<pinref part="U7" gate="G$1" pin="A"/>
 <wire x1="60.96" y1="78.74" x2="50.8" y2="78.74" width="0.1524" layer="91"/>
 </segment>
@@
 <pinref part="GND9" gate="1" pin="GND"/>
 <wire x1="-20.32" y1="101.6" x2="-20.32" y2="109.22" width="0.1524" layer="91"/>
-<pinref part="U$2" gate="G$1" pin="GND"/>
+<pinref part="IR1" gate="G$1" pin="GND"/>
 <wire x1="-20.32" y1="109.22" x2="-27.94" y2="109.22" width="0.1524" layer="91"/>
 </segment>
@@
 <wire x1="393.7" y1="22.86" x2="393.7" y2="25.4" width="0.1524" layer="91"/>
 <pinref part="GND13" gate="1" pin="GND"/>
-<pinref part="C5" gate="G$1" pin="2"/>
+<pinref part="C2" gate="G$1" pin="2"/>
 <wire x1="381" y1="30.48" x2="381" y2="25.4" width="0.1524" layer="91"/>
 <wire x1="381" y1="25.4" x2="393.7" y2="25.4" width="0.1524" layer="91"/>
@@
 </segment>
 <segment>
-<pinref part="C6" gate="G$1" pin="2"/>
+<pinref part="C3" gate="G$1" pin="2"/>
 <pinref part="GND16" gate="1" pin="GND"/>
 <wire x1="429.26" y1="45.72" x2="431.8" y2="45.72" width="0.1524" layer="91"/>
@@
 <pinref part="GND12" gate="1" pin="GND"/>
 <wire x1="396.24" y1="63.5" x2="396.24" y2="68.58" width="0.1524" layer="91"/>
-<pinref part="U$5" gate="G$1" pin="GND"/>
+<pinref part="U5" gate="G$1" pin="GND"/>
 </segment>
 <segment>
@@
 <segment>
 <pinref part="GND18" gate="1" pin="GND"/>
-<pinref part="U$1" gate="G$1" pin="3"/>
+<pinref part="SW2" gate="G$1" pin="3"/>
 <wire x1="-40.64" y1="43.18" x2="-40.64" y2="44.45" width="0.1524" layer="91"/>
-<wire x1="-40.64" y1="44.45" x2="-43.18" y2="44.45" width="0.1524" layer="91"/>
+<wire x1="-40.64" y1="44.45" x2="-55.88" y2="44.45" width="0.1524" layer="91"/>
 <junction x="-40.64" y="43.18"/>
 <pinref part="SW1" gate="A" pin="5"/>
@@
 <pinref part="P+3" gate="VCC" pin="VCC"/>
 <wire x1="60.96" y1="93.98" x2="60.96" y2="96.52" width="0.1524" layer="91"/>
-<pinref part="U$7" gate="G$1" pin="E"/>
+<pinref part="U7" gate="G$1" pin="E"/>
 <wire x1="60.96" y1="93.98" x2="50.8" y2="93.98" width="0.1524" layer="91"/>
 </segment>
@@
 </segment>
 <segment>
-<pinref part="U$2" gate="G$1" pin="VCC"/>
+<pinref part="IR1" gate="G$1" pin="VCC"/>
 <pinref part="P+8" gate="VCC" pin="VCC"/>
 <wire x1="-10.16" y1="104.14" x2="-27.94" y2="104.14" width="0.1524" layer="91"/>
@@
 <junction x="-25.4" y="50.8"/>
 <pinref part="P+11" gate="VCC" pin="VCC"/>
-<pinref part="U$1" gate="G$1" pin="1"/>
-<wire x1="-43.18" y1="46.99" x2="-43.18" y2="48.26" width="0.1524" layer="91"/>
+<pinref part="SW2" gate="G$1" pin="1"/>
+<wire x1="-55.88" y1="46.99" x2="-43.18" y2="48.26" width="0.1524" layer="91"/>
 <wire x1="-43.18" y1="48.26" x2="-25.4" y2="48.26" width="0.1524" layer="91"/>
 <pinref part="SW1" gate="A" pin="8"/>
@@
 <wire x1="411.48" y1="81.28" x2="421.64" y2="81.28" width="0.1524" layer="91"/>
 <label x="416.56" y="81.28" size="1.778" layer="95"/>
-<pinref part="U$5" gate="G$1" pin="SCL2"/>
+<pinref part="U5" gate="G$1" pin="SCL2"/>
 </segment>
 <segment>
@@
 <wire x1="411.48" y1="78.74" x2="421.64" y2="78.74" width="0.1524" layer="91"/>
 <label x="416.56" y="76.2" size="1.778" layer="95"/>
-<pinref part="U$5" gate="G$1" pin="SDA2"/>
+<pinref part="U5" gate="G$1" pin="SDA2"/>
 </segment>
 <segment>
@@
 <wire x1="66.04" y1="86.36" x2="73.66" y2="86.36" width="0.1524" layer="91"/>
 <label x="68.58" y="86.36" size="1.778" layer="95"/>
-<pinref part="U$7" gate="G$1" pin="S"/>
+<pinref part="U7" gate="G$1" pin="S"/>
 <wire x1="55.88" y1="86.36" x2="58.42" y2="86.36" width="0.1524" layer="91"/>
 <wire x1="58.42" y1="86.36" x2="58.42" y2="91.44" width="0.1524" layer="91"/>
@@
 <net name="IR_IN" class="0">
 <segment>
-<pinref part="U$2" gate="G$1" pin="OUT"/>
+<pinref part="IR1" gate="G$1" pin="OUT"/>
 <wire x1="-27.94" y1="114.3" x2="-15.24" y2="114.3" width="0.1524" layer="91"/>
 <label x="-25.4" y="114.3" size="1.778" layer="95"/>
@@
 <segment>
 <label x="-78.74" y="48.26" size="1.778" layer="95"/>
-<pinref part="U$1" gate="G$1" pin="2"/>
+<pinref part="SW2" gate="G$1" pin="2"/>
 <wire x1="-71.12" y1="48.26" x2="-81.28" y2="48.26" width="0.1524" layer="91"/>
-<wire x1="-53.34" y1="45.72" x2="-71.12" y2="45.72" width="0.1524" layer="91"/>
+<wire x1="-66.04" y1="45.72" x2="-71.12" y2="45.72" width="0.1524" layer="91"/>
 <wire x1="-71.12" y1="45.72" x2="-71.12" y2="48.26" width="0.1524" layer="91"/>
 </segment>
@@
 <pinref part="P+14" gate="G$1" pin="3.3V"/>
 <wire x1="386.08" y1="99.06" x2="393.7" y2="96.52" width="0.1524" layer="91"/>
-<pinref part="U$5" gate="G$1" pin="VCC1"/>
+<pinref part="U5" gate="G$1" pin="VCC1"/>
 <label x="388.62" y="99.06" size="1.778" layer="95"/>
 </segment>
 <segment>
-<pinref part="C6" gate="G$1" pin="1"/>
+<pinref part="C3" gate="G$1" pin="1"/>
 <pinref part="U1" gate="G$1" pin="VDD"/>
 <wire x1="429.26" y1="53.34" x2="426.72" y2="53.34" width="0.1524" layer="91"/>
@@
 <net name="5V" class="0">
 <segment>
-<pinref part="U$5" gate="G$1" pin="VCC2"/>
+<pinref part="U5" gate="G$1" pin="VCC2"/>
 <wire x1="398.78" y1="96.52" x2="398.78" y2="101.6" width="0.1524" layer="91"/>
 <pinref part="U$4" gate="G$1" pin="5V"/>
@@
 <wire x1="381" y1="81.28" x2="370.84" y2="81.28" width="0.1524" layer="91"/>
 <label x="370.84" y="81.28" size="1.778" layer="95"/>
-<pinref part="U$5" gate="G$1" pin="SCL1"/>
+<pinref part="U5" gate="G$1" pin="SCL1"/>
 </segment>
 <segment>
@@
 <wire x1="381" y1="78.74" x2="370.84" y2="78.74" width="0.1524" layer="91"/>
 <label x="370.84" y="78.74" size="1.778" layer="95"/>
-<pinref part="U$5" gate="G$1" pin="SDA1"/>
+<pinref part="U5" gate="G$1" pin="SDA1"/>
 </segment>
 <segment>
@@
 <segment>
 <pinref part="U1" gate="G$1" pin="BYP"/>
-<pinref part="C5" gate="G$1" pin="1"/>
+<pinref part="C2" gate="G$1" pin="1"/>
 <wire x1="383.54" y1="38.1" x2="381" y2="38.1" width="0.1524" layer="91"/>
 </segment>
@@
 <net name="N$27" class="0">
 <segment>
-<pinref part="U$5" gate="G$1" pin="EN"/>
+<pinref part="U5" gate="G$1" pin="EN"/>
 <pinref part="R5" gate="G$1" pin="1"/>
 <wire x1="381" y1="86.36" x2="370.84" y2="86.36" width="0.1524" layer="91"/>
