File: circuit/hackerling.sch (EAGLE design)
At the start: 41 parts, among them IC1 MCP23017SP, IC2 MCP2300X/P, IC3 MIC5219BM5, SW2 SWITCH_B13EH, U1 MMA8452Q, U2 LCD_16X2, U3 ARDUINOR3-BPLACE, U4 ACCELEROMETER, U5 PCA9306, U6 ACCELEROMETER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

Commit message: before moving pins around
Other:
- note added: "Need Resistor"
Changed lines of the file:
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@@
 <text x="2.54" y="-12.7" size="1.778" layer="209">TODO: add solder jumper</text>
 <wire x1="10.16" y1="20.32" x2="10.16" y2="-6.35" width="0.1524" layer="209"/>
+<text x="166.37" y="-13.97" size="1.778" layer="209">Need Resistor</text>
+<text x="165.1" y="-16.51" size="1.778" layer="209">Need Resistor</text>
+<text x="166.37" y="-19.05" size="1.778" layer="209">Need Resistor</text>
+<text x="7.62" y="33.02" size="1.778" layer="209">Need Resistor</text>
+<text x="5.08" y="45.72" size="1.778" layer="209">Need Resistor</text>
+<text x="158.75" y="43.18" size="1.778" layer="209">Need Resistor</text>
+<text x="158.75" y="48.26" size="1.778" layer="209">Need Resistor</text>
+<text x="158.75" y="50.8" size="1.778" layer="209">Need Resistor</text>
+<text x="158.75" y="53.34" size="1.778" layer="209">Need Resistor</text>
 </plain>
 <instances>
